File: mosfet_dut_rev1.kicad_sch (KiCad schematic)
At the start: 45 parts, among them J1 USB_C_Receptacle_USB2.0_16P, J2 Conn_01x02, J3 Conn_01x02, J4 Conn_01x02, J5 Conn_01x02, J6 Conn_01x02, Q1 AO3400A, Q2 AO3400A, Q3 AO3400A, Q4 AO3400A, SW1 SW_Push, U1 USBLC6-2SC6, U2 ME6211C33M5, U3 CH340C, U4 ESP32-WROOM-32E, U5 74HC4051, U6 INA219AxD

Commit message: Rev 1.2 Final
Parts:
- removed C4: 0.1uF, Capacitor_SMD:C_0603_1608Metric, symbol Device:C
- removed C5, C7: 0.1uF, Capacitor_SMD:C_0603_1608Metric, symbol Device:C_Small
- removed C6: 10uF, Capacitor_SMD:C_0603_1608Metric, symbol Device:C_Small
- removed R3, R4: 5k1, Resistor_SMD:R_0603_1608Metric, symbol Device:R
- removed U2: ME6211C33M5, Package_TO_SOT_SMD:SOT-23-5, symbol Regulator_Linear:ME6211C33M5
- removed U3: CH340C, Package_SO:SOIC-16_3.9x9.9mm_P1.27mm, symbol Interface_USB:CH340C
- removed U4: ESP32-WROOM-32E, RF_Module:ESP32-WROOM-32E, symbol RF_Module:ESP32-WROOM-32E
- removed U5: 74HC4051, Package_SO:SO-16_3.9x9.9mm_P1.27mm, symbol 74xx:74HC4051
- removed U6: INA219AxD, Package_SO:SOIC-8_3.9x4.9mm_P1.27mm, symbol Sensor_Energy:INA219AxD
- added C10, C11, C6, C8, C9: 0.1uF, Capacitor_SMD:C_0603_1608Metric, symbol Device:C
- added C4, C5: 10uF, Capacitor_Tantalum_SMD:CP_EIA-3216-18_Kemet-A, symbol Device:C_Polarized
- added C7: 1uF, Capacitor_SMD:C_0603_1608Metric, symbol Device:C
- added D1: LED_R, LED_SMD:LED_0805_2012Metric, symbol Device:LED
- added D2, D3, D4, D5, D6: LED_G, LED_SMD:LED_0805_2012Metric, symbol Device:LED
- added R10, R17, R8: 2m, Resistor_SMD:R_2512_6332Metric, symbol Device:R
- added R16, R21, R23: 100k, Resistor_SMD:R_0603_1608Metric, symbol Device:R
- added R18, R19, R6, R7: 1k, Resistor_SMD:R_0603_1608Metric, symbol Device:R
- added R9: 5k1, Resistor_SMD:R_0603_1608Metric, symbol Device:R
- added U1, U4, U6, U7: INA226, Package_SO:VSSOP-10_3x3mm_P0.5mm, symbol Sensor_Energy:INA226
- added U2: AMS1117-3.3, Package_TO_SOT_SMD:SOT-223-3_TabPin2, symbol Regulator_Linear:AMS1117-3.3
- added U5: ESP32-C3-WROOM-02, RF_Module:ESP32-C3-WROOM-02, symbol RF_Module:ESP32-C3-WROOM-02
- C2: value 1uF -> 0.1uF; JLCPCB Part # CL10A105KB8NNNC -> C14663
- FID1, FID2, FID3: now left out of the parts list
- J1: renamed from J2; value Conn_01x02 -> SCREW_TERMINAL; now fitted
- J3, J6: value Conn_01x02 -> SCREW_TERMINAL; now fitted
- J4: renamed from J5; value Conn_01x02 -> SCREW_TERMINAL; now fitted
- J5: renamed from J4; value Conn_01x02 -> SCREW_TERMINAL; now fitted
- R11, R12: value 50m -> 1k; footprint Resistor_SMD:R_2512_6332Metric -> Resistor_SMD:R_0603_1608Metric; JLCPCB Part # C7420008 -> C21190; MPN YAGEO RL2512FK-070R05L -> (none)
- R13: value 50m -> 5k1; footprint Resistor_SMD:R_2512_6332Metric -> Resistor_SMD:R_0603_1608Metric; JLCPCB Part # C7420008 -> C23186; MPN YAGEO RL2512FK-070R05L -> (none)
- R14: value 50m -> 100k; footprint Resistor_SMD:R_2512_6332Metric -> Resistor_SMD:R_0603_1608Metric; JLCPCB Part # C7420008 -> C25803; MPN YAGEO RL2512FK-070R05L -> (none)
- R5: value 5k1 -> 2m; footprint Resistor_SMD:R_0603_1608Metric -> Resistor_SMD:R_2512_6332Metric; JLCPCB Part # C23186 -> C2994640; MPN (none) -> HoLLR2512-3W-2mR-1%
- renumbered J1 to J2, Q3 to Q2, Q2 to Q3, R10 to R1, R7 to R15, R9 to R2, R6 to R20, R8 to R22, R1 to R3, R2 to R4, SW1 to RESET, U1 to U3
Connections:
- net UARTDDTR is gone; now on net +3V3: C3.1
- net +3V3: now also C10.1, C11.1, C4.1, C5.1, C6.1, C7.1, C8.1, R7.1, R9.1, U1.6 (VS), U2.2 (VO), U4.6 (VS), U5.1 (3V3), U6.6 (VS), U7.6 (VS)
- net +VBUS: now also U2.3 (VI)
- net GND: now also C3.2, R14.2, C10.2, C11.2, C4.2, C5.2, C6.2, C7.2, C8.2, C9.2, D1.1 (K), D2.1 (K), D3.1 (K), D4.1 (K), D5.1 (K), D6.1 (K), R16.2, R21.2, R23.2, U1.1 (A1), U1.2 (A0), U1.7 (GND), U2.1 (GND), U4.1 (A1), U4.2 (A0), U4.7 (GND), U5.19 (GND), U5.9 (GND), U6.1 (A1), U6.2 (A0), U6.7 (GND), U7.1 (A1), U7.2 (A0), U7.7 (GND); no longer R15.2, R20.2, R22.2, R5.2, RESET.1
- net I2C_SCL: now also R2.2, U1.5 (SCL), U4.5 (SCL), U5.3 (IO4), U6.5 (SCL), U7.5 (SCL); no longer R1.2
- net I2C_SDA: now also R1.2, U1.4 (SDA), U4.4 (SDA), U5.4 (IO5), U6.4 (SDA), U7.4 (SDA); no longer R2.2
- net M1_CTRL: now also R11.1, R13.2, U5.5 (IO6); no longer Q1.1 (G), R5.1
- net M2_CTRL: now also R20.2, R18.2, U5.6 (IO7); no longer Q3.1 (G), R20.1
- net M3_CTRL: now also R12.1, R15.2, U5.7 (IO8); no longer Q2.1 (G), R15.1
- net M4_CTRL: now also R22.2, R19.2, U5.8 (IO9); no longer Q4.1 (G), R22.1
- net POWER_SENSE+: now also R5.2, R10.2, R17.2, R8.2, U1.10 (Vin+), U4.10 (Vin+), U6.10 (Vin+), U7.10 (Vin+); no longer R11.2, R12.2, R13.2, R14.2
- net OUT1+ renamed DUT1+
- net DUT1+: now also R5.1, U1.8 (Vbus), U1.9 (Vin-); no longer R11.1
- net OUT1- renamed DUT1-
- net OUT2+ renamed DUT3+
- net DUT3+: now also R10.1, U6.8 (Vbus), U6.9 (Vin-); no longer R12.1
- net OUT2- renamed DUT2-
- net DUT2-: now also J4.2 (Pin_2); no longer J5.2 (Pin_2)
- net OUT3+: no longer names the net of R13.1
- net OUT3+: now also Q1.1 (G), R14.1; no longer J4.1 (Pin_1)
- net OUT3- renamed DUT3-
- net DUT3-: now also J5.2 (Pin_2); no longer J4.2 (Pin_2)
- net OUT4+ renamed DUT4+
- net DUT4+: now also R17.1, U7.8 (Vbus), U7.9 (Vin-); no longer R14.1
- net OUT4- renamed DUT4-
- net UARTDDTR_EN renamed ENABLE
- net ENABLE: now also R9.2, U5.2 (EN); no longer C3.2
- net USBD+ renamed USBC_DP
- net USBC_DP: now also U5.14 (DP_IO19)
- net USBD- renamed USBC_DN
- net USBC_DN: now also U5.13 (DM_IO18)
- new net: C9.1, RESET.1
- new net: D6.2 (A), R19.1
- new net: Q3.1 (G), R20.1, R21.1
- new net: Q4.1 (G), R22.1, R23.1
- new net: Q2.1 (G), R15.1, R16.1
- new net: D3.2 (A), R11.2
- new net: D2.2 (A), R7.2
- new net: D4.2 (A), R12.2
- new net: R6.1, U5.18 (IO0)
- new net: D1.2 (A), R6.2
- new net: D5.2 (A), R18.1
- new net DUT2+: J4.1 (Pin_1), R8.1, U4.8 (Vbus), U4.9 (Vin-)
- no-connect marks 25 -> 12
Other:
- note removed: "Current Sensor"
- note removed: "I2C Addr = 0x40"
- note removed: "USB -> UART"
- moved on the sheet: C1, FID1, FID2, FID3, H1, H2, H3, H4, J2, Q1, Q2, Q3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
